Commit message: Navigation working on tb2-1

File: turtlebot2_description/robots/icclab_tb2-1_urdf.xacro (robot description, xacro)
@@ -10,5 +10,5 @@
   <xacro:stack_hexagons parent="base_link" />
   <xacro:scanse prefix="scanse" prefix_topic="" parent="base_link" >
-   <origin xyz="0 0 0.33" rpy="3.1415 0 2.1"/>
+   <origin xyz="0 0 0.39" rpy="3.1415 0 2.1"/>
   </xacro:scanse>
 </robot>

Commit message: Added camera to tb2-1 xacro

File: turtlebot2_description/robots/icclab_tb2-1_urdf.xacro (robot description, xacro)
@@ -12,3 +12,9 @@
    <origin xyz="0 0 0.39" rpy="3.1415 0 2.1"/>
   </xacro:scanse>
+  <joint name="camera_joint" type="fixed">
+    <origin xyz="0.15 0 0.43" rpy="0 0 0"/>
+    <parent link="base_link"/>
+    <child link="camera_link"/>
+  </joint>
+  <link name="camera_link"/>
 </robot>
